Commit message: Add arm_card_dealer package and device modulebus support
- Add new arm_card_dealer package for card handling automation
- Add device/modebus module for Modbus communication with pumps and sensors
- Update a1x_hardware_bridge with joint state remapping and hardware interface
- Enhance move_to_pose with improved TF query strategies and parallel execution
- Add pilz_cartesian_limits configuration for MoveIt2
- Update ROS2 controllers and joint limits configuration
- Add run.sh with common ROS2 commands for development workflow
- Various optimizations for trajectory planning and execution

File: a1x/urdf/a1x.urdf (robot description, URDF)
Before this commit: robot a1x, 7 links, 6 joints
Joints:
- joint arm_joint2: limit lower=0 upper=3.1416 effort=50 velocity=12.5664 -> lower=-0.1 upper=3.1416 effort=50 velocity=12.5664

File: a1x_moveit_config/config/a1x.ros2_control.xacro (robot description, xacro)
@@ -5,5 +5,5 @@
         <ros2_control name="${name}" type="system">
             <hardware>
-                <!-- By default, set up controllers for simulation. This won't work on real hardware -->
+                <!-- 使用模拟硬件接口 -->
                 <plugin>mock_components/GenericSystem</plugin>
             </hardware>
